Commit message: Integrate Astra ROS observation, policy, safety and evidence gates

File: 61-embodied-agent-architecture-lab/astra_description/urdf/astra.urdf.xacro (robot description, xacro)
@@ -39,5 +39,5 @@
   <link name="camera_optical_frame"/><joint name="camera_optical_joint" type="fixed"><parent link="camera_link"/><child link="camera_optical_frame"/><origin rpy="-1.5708 0 -1.5708"/></joint>
   <xacro:simple_link name="lidar_link" mass="0.1" sx="0.07" sy="0.07" sz="0.04"/>
-  <joint name="lidar_mount" type="fixed"><parent link="base_link"/><child link="lidar_link"/><origin xyz="0 0 0.18"/></joint>
+  <joint name="lidar_mount" type="fixed"><parent link="base_link"/><child link="lidar_link"/><origin xyz="0.30 0 0.18"/></joint>
   <link name="imu_link"/><joint name="imu_mount" type="fixed"><parent link="base_link"/><child link="imu_link"/></joint>
   <link name="bumper_link"/><joint name="bumper_mount" type="fixed"><parent link="base_link"/><child link="bumper_link"/><origin xyz="0.29 0 0"/></joint>
@@ -45,4 +45,4 @@
   <gazebo reference="lidar_link"><sensor name="lidar_2d" type="gpu_lidar"><always_on>true</always_on><update_rate>10</update_rate><topic>/astra/sensors/scan</topic><lidar><scan><horizontal><samples>360</samples><min_angle>-3.14159</min_angle><max_angle>3.14159</max_angle></horizontal></scan><range><min>0.1</min><max>10.0</max></range></lidar></sensor></gazebo>
   <gazebo reference="imu_link"><sensor name="imu" type="imu"><always_on>true</always_on><update_rate>50</update_rate><topic>/astra/sensors/imu</topic></sensor></gazebo>
-  <gazebo><plugin filename="gz-sim-diff-drive-system" name="gz::sim::systems::DiffDrive"><left_joint>left_wheel_joint</left_joint><right_joint>right_wheel_joint</right_joint><wheel_separation>0.46</wheel_separation><wheel_radius>0.09</wheel_radius><topic>/astra/control/cmd_vel</topic><odom_topic>/astra/sensors/odom</odom_topic><frame_id>odom</frame_id><child_frame_id>base_link</child_frame_id></plugin></gazebo>
+  <gazebo><plugin filename="gz-sim-diff-drive-system" name="gz::sim::systems::DiffDrive"><left_joint>left_wheel_joint</left_joint><right_joint>right_wheel_joint</right_joint><wheel_separation>0.46</wheel_separation><wheel_radius>0.09</wheel_radius><topic>/astra/control/cmd_vel</topic><odom_topic>/astra/sensors/odom</odom_topic><frame_id>odom</frame_id><child_frame_id>base_link</child_frame_id><cmd_vel_timeout>0.25</cmd_vel_timeout></plugin></gazebo>
 </robot>

Commit message: Integrate Astra RGB-D perception and typed ROS skills

File: 61-embodied-agent-architecture-lab/astra_description/urdf/astra.urdf.xacro (robot description, xacro)
@@ -36,11 +36,11 @@
   <joint name="gripper_right_mount" type="fixed"><parent link="tool0"/><child link="gripper_right"/><origin xyz="0 -0.04 0.06"/></joint>
   <xacro:simple_link name="camera_link" mass="0.1" sx="0.08" sy="0.10" sz="0.04"/>
-  <joint name="camera_mount" type="fixed"><parent link="base_link"/><child link="camera_link"/><origin xyz="0.22 0 0.18"/></joint>
-  <link name="camera_optical_frame"/><joint name="camera_optical_joint" type="fixed"><parent link="camera_link"/><child link="camera_optical_frame"/><origin rpy="-1.5708 0 -1.5708"/></joint>
+  <joint name="camera_mount" type="fixed"><parent link="base_link"/><child link="camera_link"/><origin xyz="0.36 0 0.30"/></joint>
+  <link name="camera_optical_frame"/><joint name="camera_optical_joint" type="fixed"><parent link="camera_link"/><child link="camera_optical_frame"/><origin xyz="0.08 0 0" rpy="-1.5708 0 -1.5708"/></joint>
   <xacro:simple_link name="lidar_link" mass="0.1" sx="0.07" sy="0.07" sz="0.04"/>
   <joint name="lidar_mount" type="fixed"><parent link="base_link"/><child link="lidar_link"/><origin xyz="0.30 0 0.18"/></joint>
   <link name="imu_link"/><joint name="imu_mount" type="fixed"><parent link="base_link"/><child link="imu_link"/></joint>
   <link name="bumper_link"/><joint name="bumper_mount" type="fixed"><parent link="base_link"/><child link="bumper_link"/><origin xyz="0.29 0 0"/></joint>
-  <gazebo reference="camera_link"><sensor name="head_rgbd" type="rgbd_camera"><always_on>true</always_on><update_rate>15</update_rate><topic>/astra/sensors/rgbd</topic><camera><horizontal_fov>1.047</horizontal_fov><image><width>320</width><height>240</height><format>R8G8B8</format></image><clip><near>0.1</near><far>8.0</far></clip></camera></sensor></gazebo>
+  <gazebo reference="camera_link"><sensor name="head_rgbd" type="rgbd_camera"><pose>0.08 0 0 0 0 0</pose><always_on>true</always_on><update_rate>15</update_rate><topic>/astra/sensors/rgbd</topic><gz_frame_id>camera_optical_frame</gz_frame_id><camera><horizontal_fov>1.047</horizontal_fov><image><width>320</width><height>240</height><format>R8G8B8</format></image><clip><near>0.1</near><far>8.0</far></clip></camera></sensor></gazebo>
   <gazebo reference="lidar_link"><sensor name="lidar_2d" type="gpu_lidar"><always_on>true</always_on><update_rate>10</update_rate><topic>/astra/sensors/scan</topic><lidar><scan><horizontal><samples>360</samples><min_angle>-3.14159</min_angle><max_angle>3.14159</max_angle></horizontal></scan><range><min>0.1</min><max>10.0</max></range></lidar></sensor></gazebo>
   <gazebo reference="imu_link"><sensor name="imu" type="imu"><always_on>true</always_on><update_rate>50</update_rate><topic>/astra/sensors/imu</topic></sensor></gazebo>

Commit message: Integrate Gazebo six-axis arm controllers

File: 61-embodied-agent-architecture-lab/astra_description/urdf/astra.urdf.xacro (robot description, xacro)
@@ -1,4 +1,5 @@
 <?xml version="1.0"?>
 <robot xmlns:xacro="http://www.ros.org/wiki/xacro" name="astra_synthetic_v1">
+  <xacro:arg name="controllers_file" default="$(find astra_description)/config/controllers.yaml"/>
   <xacro:macro name="simple_link" params="name mass sx sy sz">
     <link name="${name}">
@@ -42,4 +43,26 @@
   <link name="imu_link"/><joint name="imu_mount" type="fixed"><parent link="base_link"/><child link="imu_link"/></joint>
   <link name="bumper_link"/><joint name="bumper_mount" type="fixed"><parent link="base_link"/><child link="bumper_link"/><origin xyz="0.29 0 0"/></joint>
+  <xacro:macro name="arm_control" params="number">
+    <joint name="arm_joint_${number}">
+      <command_interface name="position"><param name="min">-1.5</param><param name="max">1.5</param></command_interface>
+      <state_interface name="position"><param name="initial_value">0.0</param></state_interface>
+      <state_interface name="velocity"/>
+    </joint>
+  </xacro:macro>
+  <ros2_control name="AstraArmSim" type="system">
+    <hardware><plugin>gz_ros2_control/GazeboSimSystem</plugin></hardware>
+    <xacro:arm_control number="1"/>
+    <xacro:arm_control number="2"/>
+    <xacro:arm_control number="3"/>
+    <xacro:arm_control number="4"/>
+    <xacro:arm_control number="5"/>
+    <xacro:arm_control number="6"/>
+  </ros2_control>
+  <gazebo>
+    <plugin filename="libgz_ros2_control-system.so" name="gz_ros2_control::GazeboSimROS2ControlPlugin">
+      <parameters>$(arg controllers_file)</parameters>
+      <ros><remapping>/robot_description:=/astra/robot_description</remapping></ros>
+    </plugin>
+  </gazebo>
   <gazebo reference="camera_link"><sensor name="head_rgbd" type="rgbd_camera"><pose>0.08 0 0 0 0 0</pose><always_on>true</always_on><update_rate>15</update_rate><topic>/astra/sensors/rgbd</topic><gz_frame_id>camera_optical_frame</gz_frame_id><camera><horizontal_fov>1.047</horizontal_fov><image><width>320</width><height>240</height><format>R8G8B8</format></image><clip><near>0.1</near><far>8.0</far></clip></camera></sensor></gazebo>
   <gazebo reference="lidar_link"><sensor name="lidar_2d" type="gpu_lidar"><always_on>true</always_on><update_rate>10</update_rate><topic>/astra/sensors/scan</topic><lidar><scan><horizontal><samples>360</samples><min_angle>-3.14159</min_angle><max_angle>3.14159</max_angle></horizontal></scan><range><min>0.1</min><max>10.0</max></range></lidar></sensor></gazebo>
